File: kicad/Raspberry Pi Fan Hat.sch (KiCad schematic (older format))
At the start: 5 parts, among them J1 Conn_01x03_Female, J2 Conn_01x02_Male, Q1 BC817

Commit message: Added data for kicost
Parts:
- D1: manf# (none) -> TS4148C RZG
- J1: manf# (none) -> RND 205-00643
- J2: manf# (none) -> SL 1X36W 2,54
- Q1: manf# (none) -> BC817-25
- R1: manf# (none) -> RND1550805S8F4300T5E
Changed lines of the file:
@@
 F 2 "Connector_PinSocket_2.54mm:PinSocket_1x03_P2.54mm_Vertical" H 1200 1375 50  0001 C CNN
 F 3 "~" H 1200 1375 50  0001 C CNN
+F 4 "RND 205-00643" H 1200 1375 50  0001 C CNN "manf#"
 	1    1200 1375
 	-1   0    0    -1
@@
 F 2 "Connector_PinHeader_2.54mm:PinHeader_1x02_P2.54mm_Horizontal" H 1200 2300 50  0001 C CNN
 F 3 "~" H 1200 2300 50  0001 C CNN
+F 4 "SL 1X36W 2,54" H 1200 2300 50  0001 C CNN "manf#"
 	1    1200 2300
 	1    0    0    1
@@
 F 2 "Package_TO_SOT_SMD:SOT-23" H 3625 1300 50  0001 L CIN
 F 3 "http://www.fairchildsemi.com/ds/BC/BC817.pdf" H 3425 1375 50  0001 L CNN
+F 4 "BC817-25" H 3425 1375 50  0001 C CNN "manf#"
 	1    3425 1375
 	1    0    0    -1
@@
 F 2 "Resistor_SMD:R_0805_2012Metric_Pad1.15x1.40mm_HandSolder" V 3005 1375 50  0001 C CNN
 F 3 "~" H 3075 1375 50  0001 C CNN
+F 4 "RND1550805S8F4300T5E" H 3075 1375 50  0001 C CNN "manf#"
 	1    3075 1375
 	0    1    1    0
@@
 F 2 "Resistor_SMD:R_0603_1608Metric_Pad1.05x0.95mm_HandSolder" H 1600 2150 50  0001 C CNN
 F 3 "~" H 1600 2150 50  0001 C CNN
+F 4 "TS4148C RZG" H 1600 2150 50  0001 C CNN "manf#"
 	1    1600 2150
 	0    1    1    0
